File: Hardware/precond/_autosave-precond.kicad_sch (KiCad schematic)
At the start: 29 parts, among them J1 Conn_Coaxial, J2 Conn_Coaxial, J3 Buck_logic_in, J4 3.3V_header, Q1 PMOS, U1 OPA2340, U2 OPA2340

Commit message: stuff
Parts:
- added R5: 1k, symbol Device:R
Connections:
- net +5V: now also R5.1
- net at Q1.2 (G): now also R5.2; no longer J3.1 (Pin_1)
Other:
- moved on the sheet: J3
