File: Hardware/precond/pcb_old.kicad_pcb (KiCad board)
At the start: 2 copper layers, 90 x 97.5 mm, 40 parts, among them J1 Conn_Coaxial, J2 Conn_Coaxial, J3 Buck_logic_in, J4 3.3V_header, J5 XADC_headder, J6 Pmod_to_UART, Q1 IRLML6344TRPBF, Q2 IRLML9301TRPBF, U1 OPA2340, U2 OPA2340

Commit message: yanis do the thing you wanted i left the header and microcontroller for you on top
Parts:
- moved J5 113.8 mm to (46.3, 142.4)
- moved J6 94.5 mm to (48.4, 133.0)
- moved C6 72.1 mm to (129.8, 73.0), turned to -90 degrees
- moved J3 64.9 mm to (129.2, 87.0), turned to 90 degrees
- moved A1 64.8 mm to (34.6, 154.9), turned to 180 degrees
- moved C2 59.1 mm to (121.5, 86.2), turned to 90 degrees
- moved D3 58.8 mm to (115.0, 90.8), turned to 0 degrees
- moved J4 57.8 mm to (55.0, 159.2)
- moved R7 56.5 mm to (118.9, 86.1)
- moved R6 55.1 mm to (123.9, 86.1)
- moved L1 55.0 mm to (108.2, 90.8), turned to 90 degrees
- moved Q1 53.3 mm to (124.8, 81.7), turned to 90 degrees
- moved Rf2 51.7 mm to (113.9, 105.0), turned to 180 degrees
- moved R8 50.1 mm to (116.5, 86.1)
- moved R3 49.5 mm to (127.6, 96.5), turned to 180 degrees
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Routing:
- net +5V: track 102.1 -> 0.00 mm, vias 1 -> 0
- net +3.3V: track 130.5 -> 49.8 mm
- net /Op1_out: track 69.9 -> 5.78 mm
- net /Op2_out: track 58.3 -> 9.57 mm
- net Net-(D3-K): track 50.8 -> 17.6 mm, vias 2 -> 0
- net Net-(D10-A): track 47.3 -> 15.0 mm, vias 2 -> 0
- net Net-(D8-A): track 49.5 -> 22.0 mm, vias 2 -> 0
- net GND: track 10.5 -> 0.00 mm
- net Net-(A1-GPIO16): track 7.77 -> 0.00 mm
- net Net-(D5-A1): track 15.5 -> 7.94 mm
- net Net-(A1-GPIO17): track 7.54 -> 0.00 mm
- net Net-(D1-A1): track 15.6 -> 9.16 mm
- net Net-(J1-In): track 10.8 -> 4.76 mm
- net Net-(U1B-+): track 11.2 -> 7.26 mm
- net /Op0.5V_1: track 17.3 -> 13.7 mm
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Other:
- outline, holes or cut-outs redrawn
